Commit message: add semantic sensor to agents & habitat_mas_agents configs

File: habitat-mas/habitat_mas/data/robot_urdf/dji_m100_sensors_scaled_default.urdf (robot description, URDF)
Before this commit: robot dji_m100, 10 links, 9 joints
Links:
- removed link head
- added link head_camera, mass 1.0
Joints:
- joint head_joint: child head -> head_camera

File: habitat-mas/habitat_mas/data/robot_urdf/hab_fetch_arm_only.urdf (robot description, URDF)
Before this commit: robot fetch, 27 links, 26 joints
Links:
- removed link articulated_agent_arm
- added link articulated_agent_arm_camera, mass 1.0
Joints:
- joint articulated_agent_arm_joint: child articulated_agent_arm -> articulated_agent_arm_camera

File: habitat-mas/habitat_mas/data/robot_urdf/hab_fetch_default.urdf (robot description, URDF)
Before this commit: robot fetch, 28 links, 27 joints
Links:
- removed link articulated_agent_arm
- removed link head
- added link articulated_agent_arm_camera, mass 1.0
- added link head_camera, mass 1.0
Joints:
- joint articulated_agent_arm_joint: child articulated_agent_arm -> articulated_agent_arm_camera
- joint head_joint: child head -> head_camera

File: habitat-mas/habitat_mas/data/robot_urdf/hab_fetch_head_only.urdf (robot description, URDF)
Before this commit: robot fetch, 27 links, 26 joints
Links:
- removed link head
- added link head_camera, mass 1.0
Joints:
- joint head_joint: child head -> head_camera

File: habitat-mas/habitat_mas/data/robot_urdf/hab_spot_arm_arm_only.urdf (robot description, URDF)
Before this commit: robot spot, 24 links, 23 joints
Links:
- removed link articulated_agent_arm_depth
- removed link articulated_agent_arm_panoptic
- removed link articulated_agent_arm_rgb
- added link articulated_agent_arm_camera, mass 1.0
Joints:
- removed joint articulated_agent_arm_depth_joint
- removed joint articulated_agent_arm_panoptic_joint
- removed joint articulated_agent_arm_rgb_joint
- added joint articulated_agent_arm_joint: type fixed, parent arm0.link_wr1, child articulated_agent_arm_camera, origin xyz=-7.256090395202364e-09 -0.01799999177455902 -0.16599999368190765 rpy=0.0 -0.0 0.0, axis 1. 0. 0.

File: habitat-mas/habitat_mas/data/robot_urdf/hab_spot_arm_default.urdf (robot description, URDF)
Before this commit: robot spot, 26 links, 25 joints
Links:
- removed link articulated_agent_arm_depth
- removed link articulated_agent_arm_panoptic
- removed link articulated_agent_arm_rgb
- removed link head_stereo_left
- removed link head_stereo_right
- added link articulated_agent_arm_camera, mass 1.0
- added link head_camera, mass 1.0
Joints:
- removed joint articulated_agent_arm_depth_joint
- removed joint articulated_agent_arm_panoptic_joint
- removed joint articulated_agent_arm_rgb_joint
- removed joint head_stereo_left_joint
- removed joint head_stereo_right_joint
- added joint articulated_agent_arm_joint: type fixed, parent arm0.link_wr1, child articulated_agent_arm_camera, origin xyz=-7.256090395202364e-09 -0.01799999177455902 -0.16599999368190765 rpy=0.0 -0.0 0.0, axis 1. 0. 0.
- added joint head_joint: type fixed, parent base, child head_camera, origin xyz=0.41648226976394653 0.0 0.0 rpy=0.0 -0.0 0.0, axis 1. 0. 0.

File: habitat-mas/habitat_mas/data/robot_urdf/hab_spot_arm_head_only.urdf (robot description, URDF)
Before this commit: robot spot, 23 links, 22 joints
Links:
- removed link head_stereo_left
- removed link head_stereo_right
- added link head_camera, mass 1.0
Joints:
- removed joint head_stereo_left_joint
- removed joint head_stereo_right_joint
- added joint head_joint: type fixed, parent base, child head_camera, origin xyz=0.41648226976394653 0.0 0.0 rpy=0.0 -0.0 0.0, axis 1. 0. 0.

File: habitat-mas/habitat_mas/data/robot_urdf/hab_stretch_default.urdf (robot description, URDF)
Before this commit: robot stretch_description, 45 links, 44 joints
Links:
- removed link head
- added link head_camera, mass 1.0
Joints:
- joint head_joint: child head -> head_camera
